Commit message: fix_the_error

File: ur_description/urdf/ur5e/robotiq.ros2_control.xacro (robot description, xacro)
@@ -22,21 +22,18 @@
         <joint name="${joint_name}">
           <!-- Set PID or position interface depending on configuration -->
-          <param name="mimic">${mimicing_joint}</param>
+          <!-- <param name="mimic">${mimicing_joint}</param>
           <param name="multiplier">${multiplier}</param>
           <xacro:if value="${using_position_pid}">
-            <!-- Use position_pid interface -->
-            <param name="position_kp">3000</param>
-            <param name="position_ki">1</param>
-            <param name="position_kd">100</param>
-            <param name="position_i_max">10000</param>
+            <param name="position_kp">120</param>
+            <param name="position_ki">0</param>
+            <param name="position_kd">0.1</param>
+            <param name="position_i_max">1</param>
             <command_interface name="position_pid" />
           </xacro:if>
           <xacro:unless value="${using_position_pid}">
-            <!-- Non-PID interface depends on hardware type -->
             <xacro:unless value="${ros2_control_hardware_type == 'mujoco'}">
               <command_interface name="position" />
             </xacro:unless>
             <xacro:if value="${ros2_control_hardware_type == 'mujoco'}">
-              <!-- Also apply PID gains even if not using full PID controller -->
               <param name="position_kp">3000</param>
               <param name="position_ki">1</param>
@@ -45,4 +42,16 @@
               <command_interface name="position_pid" />
             </xacro:if>
+          </xacro:unless> -->
+           <param name="mimic">${mimicing_joint}</param>
+          <param name="multiplier">${multiplier}</param>
+          <xacro:if value="${using_position_pid}">
+            <param name="position_kp">120</param>
+            <param name="position_ki">0.0</param>
+            <param name="position_kd">0.1</param>
+            <param name="position_i_max">1</param>
+            <command_interface name="position_pid" />
+          </xacro:if>
+          <xacro:unless value="${using_position_pid}">
+            <command_interface name="position" />
           </xacro:unless>
           <state_interface name="position"/>
@@ -62,11 +71,11 @@
       </joint>
       <xacro:configure_joint joint_name="${tf_prefix}robotiq_85_left_inner_knuckle_joint"
-        mimicing_joint="${tf_prefix}robotiq_85_left_knuckle_joint" multiplier="0" />
+        mimicing_joint="${tf_prefix}robotiq_85_left_knuckle_joint" multiplier="1" />
       <xacro:configure_joint joint_name="${tf_prefix}robotiq_85_left_finger_tip_joint"
         mimicing_joint="${tf_prefix}robotiq_85_left_knuckle_joint" multiplier="-1" />
       <xacro:configure_joint joint_name="${tf_prefix}robotiq_85_right_knuckle_joint"
-        mimicing_joint="${tf_prefix}robotiq_85_left_knuckle_joint" multiplier="0" />
+        mimicing_joint="${tf_prefix}robotiq_85_left_knuckle_joint" multiplier="1" />
       <xacro:configure_joint joint_name="${tf_prefix}robotiq_85_right_inner_knuckle_joint"
-        mimicing_joint="${tf_prefix}robotiq_85_left_knuckle_joint" multiplier="0" />
+        mimicing_joint="${tf_prefix}robotiq_85_left_knuckle_joint" multiplier="1" />
       <xacro:configure_joint joint_name="${tf_prefix}robotiq_85_right_finger_tip_joint"
         mimicing_joint="${tf_prefix}robotiq_85_left_knuckle_joint" multiplier="-1" />

File: ur_description/urdf/ur5e/ur5e.ros2_control.xacro (robot description, xacro)
@@ -35,5 +35,5 @@
           </state_interface>
           <state_interface name="velocity">
-            <param name="initial_value">0.0</param>
+            <!-- <param name="initial_value">0.0</param> -->
           </state_interface>
         </joint>

File: ur_description/urdf/ur5e/ur5e_macro.xacro (robot description, xacro)
@@ -44,5 +44,5 @@
       <visual>
         <geometry>
-          <mesh filename="$(find mujoco_ros2_ur)/ur_description/meshes/ur5e/visual/base.dae" />
+          <mesh filename="package://mujoco_ros2_ur/ur_description/meshes/ur5e/visual/base.dae" />
         </geometry>
         <material name="LightGrey">
@@ -53,5 +53,5 @@
         <geometry>
           <mesh
-            filename="$(find mujoco_ros2_ur)/ur_description/meshes/ur5e/collision/meshes/base_vis.stl" />
+            filename="package://mujoco_ros2_ur/ur_description/meshes/ur5e/collision/meshes/base_vis.stl" />
         </geometry>
       </collision>
@@ -73,5 +73,5 @@
       <visual>
         <geometry>
-          <mesh filename="$(find mujoco_ros2_ur)/ur_description/meshes/ur5e/visual/shoulder.dae" />
+          <mesh filename="package://mujoco_ros2_ur/ur_description/meshes/ur5e/visual/shoulder.dae" />
         </geometry>
         <material name="LightGrey">
@@ -82,5 +82,5 @@
         <geometry>
           <mesh
-            filename="$(find mujoco_ros2_ur)/ur_description/meshes/ur5e/collision/meshes/shoulder_vis.stl" />
+            filename="package://mujoco_ros2_ur/ur_description/meshes/ur5e/collision/meshes/shoulder_vis.stl" />
         </geometry>
       </collision>
@@ -103,5 +103,5 @@
       <visual>
         <geometry>
-          <mesh filename="$(find mujoco_ros2_ur)/ur_description/meshes/ur5e/visual/upperarm.dae" />
+          <mesh filename="package://mujoco_ros2_ur/ur_description/meshes/ur5e/visual/upperarm.dae" />
         </geometry>
         <material name="LightGrey">
@@ -112,5 +112,5 @@
         <geometry>
           <mesh
-            filename="$(find mujoco_ros2_ur)/ur_description/meshes/ur5e/collision/meshes/upperarm_vis.stl" />
+            filename="package://mujoco_ros2_ur/ur_description/meshes/ur5e/collision/meshes/upperarm_vis.stl" />
         </geometry>
       </collision>
@@ -133,5 +133,5 @@
       <visual>
         <geometry>
-          <mesh filename="$(find mujoco_ros2_ur)/ur_description/meshes/ur5e/visual/forearm.dae" />
+          <mesh filename="package://mujoco_ros2_ur/ur_description/meshes/ur5e/visual/forearm.dae" />
         </geometry>
         <material name="LightGrey">
@@ -142,5 +142,5 @@
         <geometry>
           <mesh
-            filename="$(find mujoco_ros2_ur)/ur_description/meshes/ur5e/collision/meshes/forearm_vis.stl" />
+            filename="package://mujoco_ros2_ur/ur_description/meshes/ur5e/collision/meshes/forearm_vis.stl" />
         </geometry>
       </collision>
@@ -163,5 +163,5 @@
       <visual>
         <geometry>
-          <mesh filename="$(find mujoco_ros2_ur)/ur_description/meshes/ur5e/visual/wrist1.dae" />
+          <mesh filename="package://mujoco_ros2_ur/ur_description/meshes/ur5e/visual/wrist1.dae" />
         </geometry>
         <material name="LightGrey">
@@ -172,5 +172,5 @@
         <geometry>
           <mesh
-            filename="$(find mujoco_ros2_ur)/ur_description/meshes/ur5e/collision/meshes/wrist1_vis.stl" />
+            filename="package://mujoco_ros2_ur/ur_description/meshes/ur5e/collision/meshes/wrist1_vis.stl" />
         </geometry>
       </collision>
@@ -193,5 +193,5 @@
       <visual>
         <geometry>
-          <mesh filename="$(find mujoco_ros2_ur)/ur_description/meshes/ur5e/visual/wrist2.dae" />
+          <mesh filename="package://mujoco_ros2_ur/ur_description/meshes/ur5e/visual/wrist2.dae" />
         </geometry>
         <material name="LightGrey">
@@ -202,5 +202,5 @@
         <geometry>
           <mesh
-            filename="$(find mujoco_ros2_ur)/ur_description/meshes/ur5e/collision/meshes/wrist2_vis.stl" />
+            filename="package://mujoco_ros2_ur/ur_description/meshes/ur5e/collision/meshes/wrist2_vis.stl" />
         </geometry>
       </collision>
@@ -223,5 +223,5 @@
       <visual>
         <geometry>
-          <mesh filename="$(find mujoco_ros2_ur)/ur_description/meshes/ur5e/visual/wrist3.dae" />
+          <mesh filename="package://mujoco_ros2_ur/ur_description/meshes/ur5e/visual/wrist3.dae" />
         </geometry>
         <material name="LightGrey">
@@ -232,5 +232,5 @@
         <geometry>
           <mesh
-            filename="$(find mujoco_ros2_ur)/ur_description/meshes/ur5e/collision/meshes/wrist3_vis.stl" />
+            filename="package://mujoco_ros2_ur/ur_description/meshes/ur5e/collision/meshes/wrist3_vis.stl" />
         </geometry>
       </collision>
@@ -328,11 +328,11 @@
         <geometry>
           <mesh
-            filename="$(find mujoco_ros2_ur)/ur_description/urdf/ur5e/robotiq/robotiq_description/meshes/visual/robotiq_85_base_link.dae" />
-        </geometry>
-      </visual>
-      <collision>
-        <geometry>
-          <mesh
-            filename="$(find mujoco_ros2_ur)/ur_description/urdf/ur5e/robotiq/robotiq_description/meshes/collision/robotiq_85_base_link.stl" />
+            filename="package://mujoco_ros2_ur/ur_description/urdf/ur5e/robotiq/robotiq_description/meshes/visual/robotiq_85_base_link.dae" />
+        </geometry>
+      </visual>
+      <collision>
+        <geometry>
+          <mesh
+            filename="package://mujoco_ros2_ur/ur_description/urdf/ur5e/robotiq/robotiq_description/meshes/collision/robotiq_85_base_link.stl" />
         </geometry>
       </collision>
@@ -364,11 +364,11 @@
         <geometry>
           <mesh
-            filename="$(find mujoco_ros2_ur)/ur_description/urdf/ur5e/robotiq/robotiq_description/meshes/visual/robotiq_85_knuckle_link.dae" />
-        </geometry>
-      </visual>
-      <collision>
-        <geometry>
-          <mesh
-            filename="$(find mujoco_ros2_ur)/ur_description/urdf/ur5e/robotiq/robotiq_description/meshes/collision/robotiq_85_knuckle_link.stl" />
+            filename="package://mujoco_ros2_ur/ur_description/urdf/ur5e/robotiq/robotiq_description/meshes/visual/robotiq_85_knuckle_link.dae" />
+        </geometry>
+      </visual>
+      <collision>
+        <geometry>
+          <mesh
+            filename="package://mujoco_ros2_ur/ur_description/urdf/ur5e/robotiq/robotiq_description/meshes/collision/robotiq_85_knuckle_link.stl" />
         </geometry>
       </collision>
@@ -385,11 +385,11 @@
         <geometry>
           <mesh
-            filename="$(find mujoco_ros2_ur)/ur_description/urdf/ur5e/robotiq/robotiq_description/meshes/visual/robotiq_85_knuckle_link.dae" />
-        </geometry>
-      </visual>
-      <collision>
-        <geometry>
-          <mesh
-            filename="$(find mujoco_ros2_ur)/ur_description/urdf/ur5e/robotiq/robotiq_description/meshes/collision/robotiq_85_knuckle_link.stl" />
+            filename="package://mujoco_ros2_ur/ur_description/urdf/ur5e/robotiq/robotiq_description/meshes/visual/robotiq_85_knuckle_link.dae" />
+        </geometry>
+      </visual>
+      <collision>
+        <geometry>
+          <mesh
+            filename="package://mujoco_ros2_ur/ur_description/urdf/ur5e/robotiq/robotiq_description/meshes/collision/robotiq_85_knuckle_link.stl" />
         </geometry>
       </collision>
@@ -416,11 +416,11 @@
         <geometry>
           <mesh
-            filename="$(find mujoco_ros2_ur)/ur_description/urdf/ur5e/robotiq/robotiq_description/meshes/visual/robotiq_85_finger_link.dae" />
-        </geometry>
-      </visual>
-      <collision>
-        <geometry>
-          <mesh
-            filename="$(find mujoco_ros2_ur)/ur_description/urdf/ur5e/robotiq/robotiq_description/meshes/collision/robotiq_85_finger_link.stl" />
+            filename="package://mujoco_ros2_ur/ur_description/urdf/ur5e/robotiq/robotiq_description/meshes/visual/robotiq_85_finger_link.dae" />
+        </geometry>
+      </visual>
+      <collision>
+        <geometry>
+          <mesh
+            filename="package://mujoco_ros2_ur/ur_description/urdf/ur5e/robotiq/robotiq_description/meshes/collision/robotiq_85_finger_link.stl" />
         </geometry>
       </collision>
@@ -437,11 +437,11 @@
         <geometry>
           <mesh
-            filename="$(find mujoco_ros2_ur)/ur_description/urdf/ur5e/robotiq/robotiq_description/meshes/visual/robotiq_85_finger_link.dae" />
-        </geometry>
-      </visual>
-      <collision>
-        <geometry>
-          <mesh
-            filename="$(find mujoco_ros2_ur)/ur_description/urdf/ur5e/robotiq/robotiq_description/meshes/collision/robotiq_85_finger_link.stl" />
+            filename="package://mujoco_ros2_ur/ur_description/urdf/ur5e/robotiq/robotiq_description/meshes/visual/robotiq_85_finger_link.dae" />
+        </geometry>
+      </visual>
+      <collision>
+        <geometry>
+          <mesh
+            filename="package://mujoco_ros2_ur/ur_description/urdf/ur5e/robotiq/robotiq_description/meshes/collision/robotiq_85_finger_link.stl" />
         </geometry>
       </collision>
@@ -474,11 +474,11 @@
         <geometry>
           <mesh
-            filename="$(find mujoco_ros2_ur)/ur_description/urdf/ur5e/robotiq/robotiq_description/meshes/visual/robotiq_85_inner_knuckle_link.dae" />
-        </geometry>
-      </visual>
-      <collision>
-        <geometry>
-          <mesh
-            filename="$(find mujoco_ros2_ur)/ur_description/urdf/ur5e/robotiq/robotiq_description/meshes/collision/robotiq_85_inner_knuckle_link.stl" />
+            filename="package://mujoco_ros2_ur/ur_description/urdf/ur5e/robotiq/robotiq_description/meshes/visual/robotiq_85_inner_knuckle_link.dae" />
+        </geometry>
+      </visual>
+      <collision>
+        <geometry>
+          <mesh
+            filename="package://mujoco_ros2_ur/ur_description/urdf/ur5e/robotiq/robotiq_description/meshes/collision/robotiq_85_inner_knuckle_link.stl" />
         </geometry>
       </collision>
@@ -495,11 +495,11 @@
         <geometry>
           <mesh
-            filename="$(find mujoco_ros2_ur)/ur_description/urdf/ur5e/robotiq/robotiq_description/meshes/visual/robotiq_85_inner_knuckle_link.dae" />
-        </geometry>
-      </visual>
-      <collision>
-        <geometry>
-          <mesh
-            filename="$(find mujoco_ros2_ur)/ur_description/urdf/ur5e/robotiq/robotiq_description/meshes/collision/robotiq_85_inner_knuckle_link.stl" />
+            filename="package://mujoco_ros2_ur/ur_description/urdf/ur5e/robotiq/robotiq_description/meshes/visual/robotiq_85_inner_knuckle_link.dae" />
+        </geometry>
+      </visual>
+      <collision>
+        <geometry>
+          <mesh
+            filename="package://mujoco_ros2_ur/ur_description/urdf/ur5e/robotiq/robotiq_description/meshes/collision/robotiq_85_inner_knuckle_link.stl" />
         </geometry>
       </collision>
@@ -534,11 +534,11 @@
         <geometry>
           <mesh
-            filename="$(find mujoco_ros2_ur)/ur_description/urdf/ur5e/ur5e/robotiq/robotiq_description/meshes/visual/robotiq_85_finger_tip_link.dae" />
-        </geometry>
-      </visual>
-      <collision>
-        <geometry>
-          <mesh
-            filename="$(find mujoco_ros2_ur)/ur_description/urdf/ur5e/robotiq/robotiq_description/meshes/collision/robotiq_85_finger_tip_link.stl" />
+            filename="package://mujoco_ros2_ur/ur_description/urdf/ur5e/ur5e/robotiq/robotiq_description/meshes/visual/robotiq_85_finger_tip_link.dae" />
+        </geometry>
+      </visual>
+      <collision>
+        <geometry>
+          <mesh
+            filename="package://mujoco_ros2_ur/ur_description/urdf/ur5e/robotiq/robotiq_description/meshes/collision/robotiq_85_finger_tip_link.stl" />
         </geometry>
       </collision>
@@ -555,11 +555,11 @@
         <geometry>
           <mesh
-            filename="$(find mujoco_ros2_ur)/ur_description/urdf/ur5e/robotiq/robotiq_description/meshes/visual/robotiq_85_finger_tip_link.dae" />
-        </geometry>
-      </visual>
-      <collision>
-        <geometry>
-          <mesh
-            filename="$(find mujoco_ros2_ur)/ur_description/urdf/ur5e/robotiq/robotiq_description/meshes/collision/robotiq_85_finger_tip_link.stl" />
+            filename="package://mujoco_ros2_ur/ur_description/urdf/ur5e/robotiq/robotiq_description/meshes/visual/robotiq_85_finger_tip_link.dae" />
+        </geometry>
+      </visual>
+      <collision>
+        <geometry>
+          <mesh
+            filename="package://mujoco_ros2_ur/ur_description/urdf/ur5e/robotiq/robotiq_description/meshes/collision/robotiq_85_finger_tip_link.stl" />
         </geometry>
       </collision>
@@ -585,5 +585,5 @@
     <collision>
       <geometry>
-        <mesh filename="$(find mujoco_ros2_ur)/ur_description/meshes/ur5e/collision/meshes/peg.stl"/>
+        <mesh filename="package://mujoco_ros2_ur/ur_description/meshes/ur5e/collision/meshes/peg.stl"/>
       </geometry>
     </collision>
