Commit message: update_from_moveit_to_ros_controls

File: ur_description/urdf/ur5e/robotiq.ros2_control.xacro (robot description, xacro)
@@ -1,6 +1,18 @@
 <?xml version="1.0" encoding='utf-8'?>
 <robot xmlns:xacro="http://www.ros.org/wiki/xacro">
+  <xacro:macro name="robotiq_command_joint" params="tf_prefix">
+    <joint name="${tf_prefix}robotiq_85_left_knuckle_joint">
+      <param name="position_kp">120</param>
+      <param name="position_ki">0</param>
+      <param name="position_kd">0.1</param>
+      <param name="position_i_max">1</param>
+      <command_interface name="position"/>
+      <state_interface name="position"/>
+      <state_interface name="velocity"/>
+      <state_interface name="effort"/>
+    </joint>
+  </xacro:macro>
   <xacro:macro name="robotiq_ros2_control"
-    params="name initial_positions_file ros2_control_hardware_type tf_prefix using_position_pid:=false">
+    params="name initial_positions_file ros2_control_hardware_type tf_prefix mujoco_model:='' using_position_pid:=false">
     <xacro:property name="initial_positions"
       value="${xacro.load_yaml(initial_positions_file)['initial_positions']}" />
@@ -16,68 +28,147 @@
         </xacro:if>
         <xacro:if value="${ros2_control_hardware_type == 'mujoco'}">
-          <plugin>mujoco_ros2_control/MujocoSystem</plugin>
+          <plugin>mujoco_ros2_control/MujocoSystemInterface</plugin>
+          <param name="mujoco_model">${mujoco_model}</param>
         </xacro:if>
       </hardware>
       <xacro:macro name="configure_joint" params="joint_name mimicing_joint multiplier">
         <joint name="${joint_name}">
-          <!-- Set PID or position interface depending on configuration -->
-          <!-- <param name="mimic">${mimicing_joint}</param>
+          <param name="mimic">${mimicing_joint}</param>
           <param name="multiplier">${multiplier}</param>
-          <xacro:if value="${using_position_pid}">
+          <!-- <xacro:unless value="${ros2_control_hardware_type == 'mujoco'}">
             <param name="position_kp">120</param>
-            <param name="position_ki">0</param>
+            <param name="position_ki">0.1</param>
             <param name="position_kd">0.1</param>
-            <param name="position_i_max">1</param>
+            <param name="position_i_max">10</param>
             <command_interface name="position_pid" />
-          </xacro:if>
-          <xacro:unless value="${using_position_pid}">
-            <xacro:unless value="${ros2_control_hardware_type == 'mujoco'}">
-              <command_interface name="position" />
-            </xacro:unless>
-            <xacro:if value="${ros2_control_hardware_type == 'mujoco'}">
-              <param name="position_kp">3000</param>
-              <param name="position_ki">1</param>
-              <param name="position_kd">100</param>
-              <param name="position_i_max">10000</param>
-              <command_interface name="position_pid" />
-            </xacro:if>
           </xacro:unless> -->
-           <param name="mimic">${mimicing_joint}</param>
-          <param name="multiplier">${multiplier}</param>
-          <xacro:if value="${using_position_pid}">
-            <param name="position_kp">120</param>
-            <param name="position_ki">0.0</param>
-            <param name="position_kd">0.1</param>
-            <param name="position_i_max">1</param>
-            <command_interface name="position_pid" />
-          </xacro:if>
-          <xacro:unless value="${using_position_pid}">
+          <!-- <xacro:if value="${ros2_control_hardware_type == 'mujoco'}">
             <command_interface name="position" />
-          </xacro:unless>
-          <state_interface name="position"/>
-          <state_interface name="velocity"/>
+          </xacro:if> -->
+          <state_interface name="position">
+            <!-- <param name="initial_value">0.0</param> -->
+          </state_interface>
+          <state_interface name="velocity">
+            <!-- <param name="initial_value">0.0</param> -->
+          </state_interface>
           <state_interface name="effort"/>
         </joint>
       </xacro:macro>
-      <joint name="${tf_prefix}robotiq_85_left_knuckle_joint">
-        <param name="position_kp">120</param>
-        <param name="position_ki">0</param>
-        <param name="position_kd">0.1</param>
-        <param name="position_i_max">1</param>
-        <command_interface name="position_pid"/>
-        <state_interface name="position"/>
-        <state_interface name="velocity"/>
-        <state_interface name="effort"/>
+      <xacro:robotiq_command_joint tf_prefix="${tf_prefix}"/>
+      <!-- <joint name="${tf_prefix}robotiq_85_left_knuckle_joint">
+        <xacro:unless value="${ros2_control_hardware_type == 'mujoco'}">
+          <param name="position_kp">3000</param>
+          <param name="position_ki">1</param>
+          <param name="position_kd">100</param>
+          <param name="position_i_max">10000</param>
+          <command_interface name="position_pid" />
+        </xacro:unless>
+        <xacro:if value="${ros2_control_hardware_type == 'mujoco'}">
+          <command_interface name="position" />
+        </xacro:if>
+        <state_interface name="position">
+          <param name="initial_value">${initial_positions['robotiq_85_left_knuckle_joint']}</param>
+        </state_interface>
+        <state_interface name="velocity">
+          <param name="initial_value">0.0</param>
+        </state_interface>
       </joint>
-      <xacro:configure_joint joint_name="${tf_prefix}robotiq_85_left_inner_knuckle_joint"
-        mimicing_joint="${tf_prefix}robotiq_85_left_knuckle_joint" multiplier="1" />
-      <xacro:configure_joint joint_name="${tf_prefix}robotiq_85_left_finger_tip_joint"
-        mimicing_joint="${tf_prefix}robotiq_85_left_knuckle_joint" multiplier="-1" />
-      <xacro:configure_joint joint_name="${tf_prefix}robotiq_85_right_knuckle_joint"
-        mimicing_joint="${tf_prefix}robotiq_85_left_knuckle_joint" multiplier="1" />
-      <xacro:configure_joint joint_name="${tf_prefix}robotiq_85_right_inner_knuckle_joint"
-        mimicing_joint="${tf_prefix}robotiq_85_left_knuckle_joint" multiplier="1" />
-      <xacro:configure_joint joint_name="${tf_prefix}robotiq_85_right_finger_tip_joint"
-        mimicing_joint="${tf_prefix}robotiq_85_left_knuckle_joint" multiplier="-1" />
+      <joint name="${tf_prefix}robotiq_85_right_knuckle_joint">
+        <param name="mimic">${tf_prefix}robotiq_85_left_knuckle_joint</param>
+        <xacro:unless value="${ros2_control_hardware_type == 'mujoco'}">
+          <param name="position_kp">3000</param>
+          <param name="position_ki">1</param>
+          <param name="position_kd">100</param>
+          <param name="position_i_max">10000</param>
+          <command_interface name="position_pid" />
+        </xacro:unless>
+        <xacro:if value="${ros2_control_hardware_type == 'mujoco'}">
+          <command_interface name="position" />
+        </xacro:if>
+        <state_interface name="position">
+          <param name="initial_value">0.0</param>
+        </state_interface>
+        <state_interface name="velocity">
+          <param name="initial_value">0.0</param>
+        </state_interface>
+      </joint>
+      <joint name="${tf_prefix}robotiq_85_left_inner_knuckle_joint">
+        <param name="mimic">${tf_prefix}robotiq_85_left_knuckle_joint</param>
+        <xacro:unless value="${ros2_control_hardware_type == 'mujoco'}">
+          <param name="position_kp">3000</param>
+          <param name="position_ki">1</param>
+          <param name="position_kd">100</param>
+          <param name="position_i_max">10000</param>
+          <command_interface name="position_pid" />
+        </xacro:unless>
+        <xacro:if value="${ros2_control_hardware_type == 'mujoco'}">
+          <command_interface name="position" />
+        </xacro:if>
+        <state_interface name="position">
+          <param name="initial_value">0.0</param>
+        </state_interface>
+        <state_interface name="velocity">
+          <param name="initial_value">0.0</param>
+        </state_interface>
+      </joint>
+      <joint name="${tf_prefix}robotiq_85_right_inner_knuckle_joint">
+        <param name="mimic">${tf_prefix}robotiq_85_left_knuckle_joint</param>
+        <xacro:unless value="${ros2_control_hardware_type == 'mujoco'}">
+          <param name="position_kp">3000</param>
+          <param name="position_ki">1</param>
+          <param name="position_kd">100</param>
+          <param name="position_i_max">10000</param>
+          <command_interface name="position_pid" />
+        </xacro:unless>
+        <xacro:if value="${ros2_control_hardware_type == 'mujoco'}">
+          <command_interface name="position" />
+        </xacro:if>
+        <state_interface name="position">
+          <param name="initial_value">0.0</param>
+        </state_interface>
+        <state_interface name="velocity">
+          <param name="initial_value">0.0</param>
+        </state_interface>
+      </joint>
+      <joint name="${tf_prefix}robotiq_85_right_finger_tip_joint">
+        <param name="mimic">${tf_prefix}robotiq_85_left_knuckle_joint</param>
+        <param name="multiplier">-1</param>
+        <xacro:unless value="${ros2_control_hardware_type == 'mujoco'}">
+          <param name="position_kp">3000</param>
+          <param name="position_ki">1</param>
+          <param name="position_kd">100</param>
+          <param name="position_i_max">10000</param>
+          <command_interface name="position_pid" />
+        </xacro:unless>
+        <xacro:if value="${ros2_control_hardware_type == 'mujoco'}">
+          <command_interface name="position" />
+        </xacro:if>
+        <state_interface name="position">
+          <param name="initial_value">0.0</param>
+        </state_interface>
+        <state_interface name="velocity">
+          <param name="initial_value">0.0</param>
+        </state_interface>
+      </joint>
+      <joint name="${tf_prefix}robotiq_85_left_finger_tip_joint">
+        <param name="mimic">${tf_prefix}robotiq_85_left_knuckle_joint</param>
+        <param name="multiplier">-1</param>
+        <xacro:unless value="${ros2_control_hardware_type == 'mujoco'}">
+          <param name="position_kp">3000</param>
+          <param name="position_ki">1</param>
+          <param name="position_kd">100</param>
+          <param name="position_i_max">10000</param>
+          <command_interface name="position_pid" />
+        </xacro:unless>
+        <xacro:if value="${ros2_control_hardware_type == 'mujoco'}">
+          <command_interface name="position" />
+        </xacro:if>
+        <state_interface name="position">
+          <param name="initial_value">0.0</param>
+        </state_interface>
+        <state_interface name="velocity">
+          <param name="initial_value">0.0</param>
+        </state_interface>
+      </joint> -->
     </ros2_control>
   </xacro:macro>

File: ur_description/urdf/ur5e/ur5e.ros2_control.xacro (robot description, xacro)
@@ -1,6 +1,7 @@
 <?xml version="1.0" encoding='utf-8'?>
 <robot xmlns:xacro="http://www.ros.org/wiki/xacro">
+  <xacro:include filename="$(find mujoco_ros2_ur)/ur_description/urdf/ur5e/robotiq.ros2_control.xacro" />
   <xacro:macro name="ur5e_ros2_control"
-    params="name initial_positions_file ros2_control_hardware_type tf_prefix">
+    params="name initial_positions_file ros2_control_hardware_type tf_prefix mujoco_model:='' ft_sensor_name:='motor_fts' ft_mujoco_sensor_name:='motor' include_gripper:=true include_camera:=false">
     <xacro:property name="initial_positions"
       value="${xacro.load_yaml(initial_positions_file)['initial_positions']}" />
@@ -16,15 +17,124 @@
         </xacro:if>
         <xacro:if value="${ros2_control_hardware_type == 'mujoco'}">
-          <plugin>mujoco_ros2_control/MujocoSystem</plugin>
+          <plugin>mujoco_ros2_control/MujocoSystemInterface</plugin>
+          <param name="mujoco_model">${mujoco_model}</param>
         </xacro:if>
       </hardware>
+      <!-- <joint name="${tf_prefix}shoulder_pan_joint">
+        <xacro:if value="${ros2_control_hardware_type == 'mujoco'}">
+          <param name="position_kp">3000</param>
+          <param name="position_ki">1</param>
+          <param name="position_kd">100</param>
+          <param name="position_i_max">10000</param>
+          <command_interface name="position_pid" />
+        </xacro:if>
+        <xacro:unless value="${ros2_control_hardware_type == 'mujoco'}">
+          <command_interface name="velocity" />
+        </xacro:unless>
+        <state_interface name="position">
+          <param name="initial_value">${initial_positions['shoulder_pan_joint']}</param>
+        </state_interface>
+        <state_interface name="velocity">
+          <param name="initial_value">0.0</param>
+        </state_interface>
+      </joint>
+      <joint name="${tf_prefix}shoulder_lift_joint">
+        <xacro:if value="${ros2_control_hardware_type == 'mujoco'}">
+          <param name="position_kp">3000</param>
+          <param name="position_ki">1</param>
+          <param name="position_kd">100</param>
+          <param name="position_i_max">10000</param>
+          <command_interface name="position_pid" />
+        </xacro:if>
+        <xacro:unless value="${ros2_control_hardware_type == 'mujoco'}">
+          <command_interface name="velocity" />
+        </xacro:unless>
+        <state_interface name="position">
+          <param name="initial_value">${initial_positions['shoulder_lift_joint']}</param>
+        </state_interface>
+        <state_interface name="velocity">
+          <param name="initial_value">0.0</param>
+        </state_interface>
+      </joint>
+      <joint name="${tf_prefix}elbow_joint">
+        <xacro:if value="${ros2_control_hardware_type == 'mujoco'}">
+          <param name="position_kp">3000</param>
+          <param name="position_ki">1</param>
+          <param name="position_kd">100</param>
+          <param name="position_i_max">10000</param>
+          <command_interface name="position_pid" />
+        </xacro:if>
+        <xacro:unless value="${ros2_control_hardware_type == 'mujoco'}">
+          <command_interface name="velocity" />
+        </xacro:unless>
+        <state_interface name="position">
+          <param name="initial_value">${initial_positions['elbow_joint']}</param>
+        </state_interface>
+        <state_interface name="velocity">
+          <param name="initial_value">0.0</param>
+        </state_interface>
+      </joint>
+      <joint name="${tf_prefix}wrist_1_joint">
+        <xacro:if value="${ros2_control_hardware_type == 'mujoco'}">
+          <param name="position_kp">3000</param>
+          <param name="position_ki">1</param>
+          <param name="position_kd">100</param>
+          <param name="position_i_max">10000</param>
+          <command_interface name="position_pid" />
+        </xacro:if>
+        <xacro:unless value="${ros2_control_hardware_type == 'mujoco'}">
+          <command_interface name="velocity" />
+        </xacro:unless>
+        <state_interface name="position">
+          <param name="initial_value">${initial_positions['wrist_1_joint']}</param>
+        </state_interface>
+        <state_interface name="velocity">
+          <param name="initial_value">0.0</param>
+        </state_interface>
+      </joint>
+      <joint name="${tf_prefix}wrist_2_joint">
+        <xacro:if value="${ros2_control_hardware_type == 'mujoco'}">
+          <param name="position_kp">3000</param>
+          <param name="position_ki">1</param>
+          <param name="position_kd">100</param>
+          <param name="position_i_max">10000</param>
+          <command_interface name="position_pid" />
+        </xacro:if>
+        <xacro:unless value="${ros2_control_hardware_type == 'mujoco'}">
+          <command_interface name="velocity" />
+        </xacro:unless>
+        <state_interface name="position">
+          <param name="initial_value">${initial_positions['wrist_2_joint']}</param>
+        </state_interface>
+        <state_interface name="velocity">
+          <param name="initial_value">0.0</param>
+        </state_interface>
+      </joint>
+      <joint name="${tf_prefix}wrist_3_joint">
+        <xacro:if value="${ros2_control_hardware_type == 'mujoco'}">
+          <param name="position_kp">3000</param>
+          <param name="position_ki">1</param>
+          <param name="position_kd">100</param>
+          <param name="position_i_max">10000</param>
+          <command_interface name="position_pid" />
+        </xacro:if>
+        <xacro:unless value="${ros2_control_hardware_type == 'mujoco'}">
+          <command_interface name="velocity" />
+        </xacro:unless>
+        <state_interface name="position">
+          <param name="initial_value">${initial_positions['wrist_3_joint']}</param>
+        </state_interface>
+        <state_interface name="velocity">
+          <param name="initial_value">0.0</param>
+        </state_interface>
+      </joint> -->
       <xacro:macro name="configure_joint" params="joint_name initial_positions joint_name_wo_prefix">
         <joint name="${joint_name}">
           <xacro:if value="${ros2_control_hardware_type == 'mujoco'}">
             <param name="position_kp">3000</param>
-            <param name="position_ki">1</param>
-            <param name="position_kd">100</param>
+            <param name="position_ki">0</param>
+            <param name="position_kd">5</param>
             <param name="position_i_max">10000</param>
-            <command_interface name="position_pid" />
+            <command_interface name="position" />
           </xacro:if>
           <xacro:unless value="${ros2_control_hardware_type == 'mujoco'}">
@@ -37,4 +147,5 @@
             <!-- <param name="initial_value">0.0</param> -->
           </state_interface>
+          <state_interface name="effort"/>
         </joint>
       </xacro:macro>
@@ -45,5 +156,25 @@
       <xacro:configure_joint joint_name="${tf_prefix}wrist_2_joint"      initial_positions="${initial_positions}" joint_name_wo_prefix="wrist_2_joint"/>
       <xacro:configure_joint joint_name="${tf_prefix}wrist_3_joint"      initial_positions="${initial_positions}" joint_name_wo_prefix="wrist_3_joint"/>
-      <sensor name="${tf_prefix}motor_fts">
+      <xacro:if value="${include_gripper}">
+        <xacro:robotiq_command_joint tf_prefix="${tf_prefix}"/>
+      </xacro:if>
+      <xacro:if value="${include_camera}">
+        <joint name="${tf_prefix}camera_joint">
+          <param name="position_kp">20</param>
+          <param name="position_ki">0</param>
+          <param name="position_kd">1</param>
+          <param name="position_i_max">1</param>
+          <command_interface name="position"/>
+          <state_interface name="position">
+            <param name="initial_value">0.0</param>
+          </state_interface>
+          <state_interface name="velocity"/>
+        </joint>
+      </xacro:if>
+      <sensor name="${ft_sensor_name}">
+        <param name="mujoco_type">fts</param>
+        <param name="mujoco_sensor_name">${ft_mujoco_sensor_name}</param>
+        <param name="force_mjcf_suffix">_force</param>
+        <param name="torque_mjcf_suffix">_torque</param>
         <state_interface name="force.x" />
         <state_interface name="force.y" />

File: ur_description/urdf/ur5e/ur5e_macro.xacro (robot description, xacro)
@@ -519,5 +519,5 @@
       <!-- 0.04303959807 -->
       <limit lower="-3.14" upper="3.14" velocity="100.0" effort="0.1" />
-      <mimic joint="${tf_prefix}robotiq_85_left_knuckle_joint" multiplier="-1" />
+      <mimic joint="${tf_prefix}robotiq_85_left_knuckle_joint" multiplier="-1"/> <!--multiplier="-1" -->
     </joint>
     <joint name="${tf_prefix}robotiq_85_right_finger_tip_joint" type="continuous">
@@ -534,5 +534,5 @@
         <geometry>
           <mesh
-            filename="package://mujoco_ros2_ur/ur_description/urdf/ur5e/ur5e/robotiq/robotiq_description/meshes/visual/robotiq_85_finger_tip_link.dae" />
+            filename="package://mujoco_ros2_ur/ur_description/urdf/ur5e/robotiq/robotiq_description/meshes/visual/robotiq_85_finger_tip_link.dae" />
         </geometry>
       </visual>

File: ur_description/urdf/ur5e/ur5e_mujoco.urdf.xacro (robot description, xacro)
@@ -4,12 +4,15 @@
     <xacro:arg name="ros2_control_hardware_type" default="mujoco" />
     <xacro:arg name="tf_prefix" default="" />
+    <xacro:arg name="mujoco_model" default="$(find mujoco_ros2_ur)/ur_mujoco/ur5e/world.xml" />
     <link name="world" />
     <!-- Import ur5e urdf file -->
     <xacro:include filename="$(find mujoco_ros2_ur)/ur_description/urdf/ur5e/ur5e_macro.xacro" />
-    <xacro:ur5e name="ur5e" tf_prefix="$(arg tf_prefix)"  connected_to="world"  rpy="0 0 0"  xyz="0.0 0.0 0.1"/>
+    <xacro:ur5e name="ur5e" tf_prefix="$(arg tf_prefix)"  connected_to="world"  rpy="0 0 0"  xyz="0 -0.145 0.97"/>
     <!-- Import ur5e ros2_control description -->
+    <xacro:include filename="$(find mujoco_ros2_ur)/ur_description/urdf/ur5e/robotiq.ros2_control.xacro" />
     <xacro:include filename="$(find mujoco_ros2_ur)/ur_description/urdf/ur5e/ur5e.ros2_control.xacro" />
-    <xacro:include filename="$(find mujoco_ros2_ur)/ur_description/urdf/ur5e/robotiq.ros2_control.xacro" />
-    <xacro:ur5e_ros2_control name="UR5eFakeSystem" initial_positions_file="$(arg initial_positions_file)" ros2_control_hardware_type="$(arg ros2_control_hardware_type)" tf_prefix="$(arg tf_prefix)"/>
-    <xacro:robotiq_ros2_control name="RobotiqFakeSystem" initial_positions_file="$(arg initial_positions_file)" ros2_control_hardware_type="$(arg ros2_control_hardware_type)" tf_prefix="$(arg tf_prefix)"/>
+    <xacro:ur5e_ros2_control name="UR5eFakeSystem" initial_positions_file="$(arg initial_positions_file)" ros2_control_hardware_type="$(arg ros2_control_hardware_type)" tf_prefix="$(arg tf_prefix)" mujoco_model="$(arg mujoco_model)" ft_sensor_name="motor_fts" ft_mujoco_sensor_name="motor" include_gripper="true" include_camera="true"/>
+    <!-- Import d435i/camera file -->
+    <xacro:include filename="$(find mujoco_ros2_ur)/ur_description/urdf/ur5e/d435i_macro.xacro" />
+    <xacro:d435i name="CameraFakeSystem" tf_prefix="$(arg tf_prefix)" connected_to="world" rpy="0 3.14159265 1.570796325" xyz="0.23 0.46 2.06" mujoco_model="$(arg mujoco_model)" include_ros2_control="false"/>
 </robot>
